File: kicad/vibration-motor.kicad_sch (KiCad schematic)
At the start: 15 parts, among them IC1 DRV2625YFFT, J1 Conn_01x03, J2 Conn_01x08, J3 Conn_01x02, M1 Motor_DC, Q1 Q_NMOS_GSD

Commit message: update schematics
Parts:
- C1: value 100nF -> 50pF
Changed lines of the file:
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@@
 			)
 		)
-		(property "Value" "100nF"
+		(property "Value" "50pF"
 			(at 60.198 49.53 0)
 			(effects
